Commit message: Modified urdf

File: arhex_description/urdf/arhex.urdf (robot description, URDF)
Before this commit: robot arhex, 8 links, 7 joints
Links:
- link chassis: geometry collision mesh filename=package://arhex_description/meshes/modeel.stl; visual mesh filename=package://arhex_description/meshes/modeel.stl
Joints:
- joint left_wheel_hinge_back: origin xyz=-0.3 0.13 0.1 rpy=0 0 0 -> xyz=-0.15 0.12 0.1 rpy=0 0 0
- joint left_wheel_hinge_front: origin xyz=0.3 0.13 0.1 rpy=0 0 0 -> xyz=0.15 0.12 0.1 rpy=0 0 0
- joint left_wheel_hinge_mid: origin xyz=0 0.13 0.1 rpy=0 0 0 -> xyz=0 0.12 0.1 rpy=0 0 0
- joint right_wheel_hinge_back: origin xyz=-0.3 -0.13 0.1 rpy=0 0 0 -> xyz=-0.15 -0.12 0.1 rpy=0 0 0
- joint right_wheel_hinge_front: origin xyz=0.3 -0.13 0.1 rpy=0 0 0 -> xyz=0.15 -0.12 0.1 rpy=0 0 0
- joint right_wheel_hinge_mid: origin xyz=0 -0.13 0.1 rpy=0 0 0 -> xyz=0 -0.12 0.1 rpy=0 0 0

Commit message: Update arhex.urdf

File: arhex_description/urdf/arhex.urdf (robot description, URDF)
Before this commit: robot arhex, 8 links, 7 joints
Links:
- added link arm_1, mass 0.2; collision mesh filename=package://arhex_description/meshes/leg.stl; visual mesh filename=package://arhex_description/meshes/leg.stl
- link left_wheel_back: geometry collision mesh filename=package://arhex_description/meshes/leg.stl; visual mesh filename=package://arhex_description/meshes/leg.stl
- link left_wheel_front: geometry collision mesh filename=package://arhex_description/meshes/leg.stl; visual mesh filename=package://arhex_description/meshes/leg.stl
- link left_wheel_mid: geometry collision mesh filename=package://arhex_description/meshes/leg.stl; visual mesh filename=package://arhex_description/meshes/leg.stl
- link right_wheel_back: geometry collision mesh filename=package://arhex_description/meshes/leg.stl; visual mesh filename=package://arhex_description/meshes/leg.stl
- link right_wheel_front: geometry collision mesh filename=package://arhex_description/meshes/leg.stl; visual mesh filename=package://arhex_description/meshes/leg.stl
- link right_wheel_mid: geometry collision mesh filename=package://arhex_description/meshes/leg.stl; visual mesh filename=package://arhex_description/meshes/leg.stl
Joints:
- joint left_wheel_hinge_back: origin xyz=-0.15 0.12 0.1 rpy=0 0 0 -> xyz=-0.15 0.1095 0.1 rpy=0 0 0
- joint left_wheel_hinge_front: origin xyz=0.15 0.12 0.1 rpy=0 0 0 -> xyz=0.15 0.1095 0.1 rpy=0 0 0
- joint left_wheel_hinge_mid: origin xyz=0 0.12 0.1 rpy=0 0 0 -> xyz=0 0.1285 0.1 rpy=0 0 0
- joint right_wheel_hinge_back: origin xyz=-0.15 -0.12 0.1 rpy=0 0 0 -> xyz=-0.15 -0.1095 0.1 rpy=0 0 0
- joint right_wheel_hinge_front: origin xyz=0.15 -0.12 0.1 rpy=0 0 0 -> xyz=0.15 -0.1095 0.1 rpy=0 0 0
- joint right_wheel_hinge_mid: origin xyz=0 -0.12 0.1 rpy=0 0 0 -> xyz=0 -0.1285 0.1 rpy=0 0 0

Commit message: Update arhex.urdf

File: arhex_description/urdf/arhex.urdf (robot description, URDF)
Before this commit: robot arhex, 9 links, 7 joints
Joints:
- added joint link_1_base: type revolute, parent chassis, child link_1, origin xyz=0.075 0 0.1 rpy=0 0 0, axis 0 1 0, limit effort=10000 velocity=1000
- joint left_wheel_hinge_back: origin xyz=-0.15 0.1095 0.1 rpy=0 0 0 -> xyz=-0.21 0.1095 0.1 rpy=0 0 0
- joint left_wheel_hinge_front: origin xyz=0.15 0.1095 0.1 rpy=0 0 0 -> xyz=0.21 0.1095 0.1 rpy=0 0 0
- joint right_wheel_hinge_back: origin xyz=-0.15 -0.1095 0.1 rpy=0 0 0 -> xyz=-0.21 -0.1095 0.1 rpy=0 0 0
- joint right_wheel_hinge_front: origin xyz=0.15 -0.1095 0.1 rpy=0 0 0 -> xyz=0.21 -0.1095 0.1 rpy=0 0 0

Commit message: Add driver

File: arhex_description/urdf/arhex.urdf (robot description, URDF)
Before this commit: robot arhex, 9 links, 8 joints
Links:
- removed link arm_1
Joints:
- removed joint link_1_base

Commit message: remove old meshes

File: arhex_description/urdf/arhex.urdf (robot description, URDF)
Before this commit: robot arhex, 8 links, 7 joints
Links:
- link chassis: geometry collision mesh filename=package://arhex_description/meshes/base.stl; visual mesh filename=package://arhex_description/meshes/base.stl

Commit message: Make it walk without kissing the ground

File: arhex_description/urdf/arhex.urdf (robot description, URDF)
Before this commit: robot arhex, 8 links, 7 joints
Joints:
- joint left_wheel_hinge_back: limit effort=10000 velocity=1000 -> effort=30 velocity=4
- joint left_wheel_hinge_front: limit effort=10000 velocity=1000 -> effort=30 velocity=4
- joint left_wheel_hinge_mid: limit effort=10000 velocity=1000 -> effort=30 velocity=4
- joint right_wheel_hinge_back: limit effort=10000 velocity=1000 -> effort=30 velocity=4
- joint right_wheel_hinge_front: limit effort=10000 velocity=1000 -> effort=30 velocity=4
- joint right_wheel_hinge_mid: limit effort=10000 velocity=1000 -> effort=30 velocity=4
